File: KiCad/isa_opl2.sch (KiCad schematic (older format))
At the start: 61 parts, among them J1 AUDIO_OUT, P1 IRQ, P2 ADDR, Q1 2N3904, U1 74LS245, U2 74LS138, U3 74LS138, U4 74LS74, U5 74LS04, U6 YM3812, U7 Y3014B, U8 RC4136, U9 LM386

Commit message: Add v1.2 files
Signed-off-by: Sergey Kiselev <skiselev@gmail.com>
Parts:
- BUS1: symbol BUSPC -> isa_opl2-rescue:BUSPC
- C1, C10, C11, C2, C20, C21, C22, C23, C24, C25, C26, C3, C4, C5, C6, C7, C8, C9: symbol C -> isa_opl2-rescue:C
- C12, C13, C14, C15, C16, C17, C18, C19: symbol CP1 -> isa_opl2-rescue:CP1
- D1: symbol DIODE -> isa_opl2-rescue:DIODE
- HOLE1, HOLE2: symbol CONN_1 -> isa_opl2-rescue:CONN_1
- J1: symbol CONN_5 -> isa_opl2-rescue:CONN_5
- P1: symbol CONN_3X2 -> isa_opl2-rescue:CONN_3X2
- P2: symbol CONN_4X2 -> isa_opl2-rescue:CONN_4X2
- Q1: symbol NPN -> isa_opl2-rescue:NPN
- R1, R10, R11, R12, R13, R14, R15, R16, R17, R2, R3, R4, R5, R6, R7, R8, R9: symbol R -> isa_opl2-rescue:R
- RV1: symbol POT -> isa_opl2-rescue:POT
- U1: symbol 74LS245 -> 74ls-sergey:74LS245
- U2, U3: symbol 74LS138 -> 74ls-sergey:74LS138
- U4: symbol 74LS74 -> 74ls-sergey:74LS74
- U5: symbol 74LS04 -> 74ls-sergey:74LS04
- U6: symbol YM3812 -> controllers-sergey:YM3812
- U7: symbol Y3014B -> controllers-sergey:Y3014B
- U8: symbol RC4136 -> devices-sergey:RC4136
- U9: symbol LM386 -> devices-sergey:LM386
Connections:
- net RC1: no longer Q1.3 (C)
- net RC2: now also Q1.3 (C)
Other:
- moved on the sheet: C19, Q1, R13, R4
